Commit message: k lib integrated

File: assets/urdf/urdf_assembly_rigid_stl_collapsed.urdf (robot description, URDF)
Before this commit: robot urt_arm_collapsed, 7 links, 6 joints
Links:
- added link link6, mass 0.00033959712; visual mesh filename=../meshes_onshape_rigid_stl/Block.stl scale=1 1 1; visual mesh filename=../meshes_onshape_rigid_stl/Gripper.stl scale=1 1 1
- link link3: geometry visual mesh filename=../meshes_onshape_rigid_stl/FSA36_14_Rotor.stl scale=1 1 1; visual mesh filename=../meshes_onshape_rigid_stl/Part_1_9.stl scale=1 1 1
Joints:
- added joint revolute_6: type continuous, parent link5, child link6, origin xyz=-0.118800029 0.0404281961 3.33587926e-05 rpy=3.14158558 -0.523594 1.57079589, axis 1.66533454e-16 1 1.11022302e-16
- joint revolute_5: axis -5.55111512e-17 -1 0 -> -1.66533454e-16 -1 2.08166817e-17; origin xyz=-1.75582236e-13 -0.0285989518 0.370000124 rpy=5.30717959e-06 2.65358979e-06 -3.14159265 -> xyz=-1.74638573e-13 -0.0285989518 0.370000124 rpy=5.30717959e-06 -2.65358979e-06 3.14159265
